File: hardware/layouts/default/default.kicad_pcb (KiCad board)
At the start: 2 copper layers, 0 parts

Commit message: hardware: add pickable AmigoPro_PIM485 and JST-PH motor connectors; wire into main.ato; update fp-lib-tables; build passes and BOM includes new connectors
Parts:
- added C1: 100nF ±10% 16V X7R, Samsung_Electro_Mechanics_CL05B104KO5NNNC:C0402, F.Cu at (0.07, -32.0)
- added C2: 100nF ±10% 16V X7R, Samsung_Electro_Mechanics_CL05B104KO5NNNC:C0402, F.Cu at (-1.84, -30.0)
- added J1: , Connector_2Pin_JST_PH:JST_PH_B2B-PH-SM4-TB, F.Cu at (0.00, 0.00)
- added J2: , Connector_2Pin_JST_PH:JST_PH_B2B-PH-SM4-TB, F.Cu at (0.00, -10.0)
- added J3: , Connector_2Pin_JST_PH:JST_PH_B2B-PH-SM4-TB, F.Cu at (0.00, -20.0)
- added J4: , Connector_2Pin_JST_PH:JST_PH_B2B-PH-SM4-TB, F.Cu at (0.00, -30.0)
- added J5: , AmigoPro_PIM485:AmigoPro_PIM485, F.Cu at (0.00, -40.0)
- added LED1: , Hubei_KENTO_Elec_KT_0603G:LED0603-RD, F.Cu at (12.6, -0.01)
- added LED2: , Hubei_KENTO_Elec_KT_0603R:LED0603-RD, F.Cu at (2.50, 0.00)
- added R1: 10kΩ ±1% 62.5mW, UNI_ROYAL_0402WGF1002TCE:R0402, F.Cu at (2.22, -31.0)
- added R2: 10kΩ ±1% 62.5mW, UNI_ROYAL_0402WGF1002TCE:R0402, F.Cu at (2.22, -28.9)
- added R3: 10kΩ ±1% 62.5mW, UNI_ROYAL_0402WGF1002TCE:R0402, F.Cu at (2.22, -30.0)
- added R4: 1kΩ ±1% 62.5mW, UNI_ROYAL_0402WGF1001TCE:R0402, F.Cu at (10.0, 0.00)
- added R5: 10kΩ ±1% 62.5mW, UNI_ROYAL_0402WGF1002TCE:R0402, F.Cu at (0.00, 0.00)
- added SW1: , ALPSALPINE_SKTDLDE010:KEY-SMD_SKTDLDE010, F.Cu at (0.00, 0.00)
- added U1: , Bosch_Sensortec_BMP280:LGA-8_L2.5-W2.0-P0.65_AMP6127, F.Cu at (0.00, -30.0)
- added U2: , TI_DRV8833:TI_DRV8833, F.Cu at (0.00, 0.00)
- added U3: , TI_DRV8833:TI_DRV8833, F.Cu at (0.00, -10.0)
- added U4: , GY-91:GY-91, F.Cu at (0.00, -20.0)
- added U5: , Raspberry_Pi_Pico_2W:Raspberry_Pi_Pico_2W, F.Cu at (0.00, -30.0)
Routing:
- net (no net): track 0.00 -> 10.9 mm, vias 0 -> 3
- net CSB: track 0.00 -> 1.35 mm
- net footprint-cathode-0: track 0.00 -> 1.34 mm
- net footprint-cathode-1: track 0.00 -> 1.27 mm
- net MOSI: track 0.00 -> 1.18 mm
- net spi-SCL: track 0.00 -> 1.11 mm
