File: hardware/layouts/default/default.kicad_pcb (KiCad board)
At the start: 2 copper layers, 21 parts

Commit message: hardware/main.ato: cleanup unused nets; direct instance wiring; add UBlox NEO-6M GPS with UART0 and power; wire drv_right.SLEEP; reduce duplicate net names
Parts:
- U6: footprint Aideepen_GPS_Module:Aideepen_GPS_Module -> UBlox_NEO6M:UBlox_NEO6M
Connections:
- R2 pad 2: spi-SCL -> SCL
- U1 pad 4: spi-SCL -> SCL
- U4 pad SCL: footprint-SCL -> SCL
- U4 pad SDA: SDA -> MOSI
- U5 pad SCL: footprint-SCL -> SCL
- U5 pad SDA: SDA -> MOSI
Routing:
- net (no net): track 10.9 -> 13.2 mm
- net MOSI: track 1.18 -> 0.00 mm
- net spi-SCL: track 1.11 -> 0.00 mm
