File: hardware/layouts/default/default.kicad_pcb (KiCad board)
At the start: 2 copper layers, 21 parts

Commit message: Fix Ato paths, DRV8833 pinmap, Pico I2C/GPIO, and LED module
Connections:
- net VBAT_IN renamed power_batt_in-VCC
- net VM renamed power_5v-VCC
- net VSYS renamed power_batt_out-VCC
- net drv_left-nFAULT renamed drv_left-net-1
- net drv_right-nFAULT renamed drv_right-net-1
- net led_green_ind-power-anode renamed power_3v3-anode
- net led_red_ind-power-anode renamed power-anode
- J1 pad MP: footprint-net-0 -> footprint-net-1
- J2 pad MP: footprint-net-1 -> footprint-net-2
- J3 pad MP: footprint-net-2 -> footprint-net-3
- J4 pad MP: footprint-net-3 -> footprint-net-4
- U2 pad AIN1: drv_left-AIN1 -> drv_left-net-0
- U2 pad AIN2: drv_left-AIN2 -> drv_left-net-2
- U2 pad AOUT1: drv_left-AOUT1 -> drv_left-net-3
- U2 pad AOUT2: drv_left-AOUT2 -> drv_left-net-4
- U2 pad BIN1: drv_left-BIN1 -> drv_left-net-5
- U2 pad BIN2: drv_left-BIN2 -> drv_left-net-6
- U2 pad BOUT1: drv_left-BOUT1 -> drv_left-net-7
- U2 pad BOUT2: drv_left-BOUT2 -> drv_left-net-8
- U2 pad SLEEP: drv_left-SLEEP -> drv_left-net-9
- U3 pad AIN1: drv_right-AIN1 -> drv_right-net-0
- U3 pad AIN2: drv_right-AIN2 -> drv_right-net-2
- U3 pad AOUT1: drv_right-AOUT1 -> drv_right-net-3
- U3 pad AOUT2: drv_right-AOUT2 -> drv_right-net-4
- U3 pad BIN1: drv_right-BIN1 -> drv_right-net-5
- U3 pad BIN2: drv_right-BIN2 -> drv_right-net-6
- U3 pad BOUT1: drv_right-BOUT1 -> drv_right-net-7
- U3 pad BOUT2: drv_right-BOUT2 -> drv_right-net-8
- U3 pad SLEEP: drv_right-SLEEP -> drv_right-net-9
- U4 pad INT: INT -> footprint-net-0
