File: hardware/hardware/layouts/default/default.kicad_pcb (KiCad board)
At the start: 2 copper layers, 0 parts

Commit message: Apply Android build fixes and compose UI
Parts:
- added C1: 100nF ±10% 16V X7R, Samsung_Electro_Mechanics_CL05B104KO5NNNC:C0402, F.Cu at (10.1, -32.0)
- added C2: 100nF ±10% 16V X7R, Samsung_Electro_Mechanics_CL05B104KO5NNNC:C0402, F.Cu at (8.16, -30.0)
- added J1: , Connector_2Pin_JST_PH:JST_PH_B2B-PH-SM4-TB, F.Cu at (0.00, -40.0)
- added J2: , Connector_2Pin_JST_PH:JST_PH_B2B-PH-SM4-TB, F.Cu at (0.00, -50.0)
- added J3: , Connector_2Pin_JST_PH:JST_PH_B2B-PH-SM4-TB, F.Cu at (0.00, -60.0)
- added J4: , Connector_2Pin_JST_PH:JST_PH_B2B-PH-SM4-TB, F.Cu at (0.00, -70.0)
- added J5: , AmigoPro_PIM485:AmigoPro_PIM485, F.Cu at (0.00, -90.0)
- added LED1: , Hubei_KENTO_Elec_KT_0603G:LED0603-RD, F.Cu at (32.6, -0.01)
- added LED2: , Hubei_KENTO_Elec_KT_0603R:LED0603-RD, F.Cu at (52.5, 0.00)
- added R1: 10kΩ ±1% 62.5mW, UNI_ROYAL_0402WGF1002TCE:R0402, F.Cu at (12.2, -31.0)
- added R2: 10kΩ ±1% 62.5mW, UNI_ROYAL_0402WGF1002TCE:R0402, F.Cu at (12.2, -28.9)
- added R3: 10kΩ ±1% 62.5mW, UNI_ROYAL_0402WGF1002TCE:R0402, F.Cu at (12.2, -30.0)
- added R4: 1kΩ ±1% 62.5mW, UNI_ROYAL_0402WGF1001TCE:R0402, F.Cu at (30.0, 0.00)
- added R5: 10kΩ ±1% 62.5mW, UNI_ROYAL_0402WGF1002TCE:R0402, F.Cu at (50.0, 0.00)
- added SW1: , ALPSALPINE_SKTDLDE010:KEY-SMD_SKTDLDE010, F.Cu at (20.0, 0.00)
- added U1: , Bosch_Sensortec_BMP280:LGA-8_L2.5-W2.0-P0.65_AMP6127, F.Cu at (10.0, -30.0)
- added U2: , TI_DRV8833:TI_DRV8833, F.Cu at (0.00, 0.00)
- added U3: , TI_DRV8833:TI_DRV8833, F.Cu at (0.00, -10.0)
- added U4: , UBlox_NEO6M:UBlox_NEO6M, F.Cu at (0.00, -20.0)
- added U5: , GY-91:GY-91, F.Cu at (0.00, -30.0)
- added U6: , Raspberry_Pi_Pico_2W:Raspberry_Pi_Pico_2W, F.Cu at (0.00, -80.0)
Routing:
- net power_3v3-anode: track 0.00 -> 6.88 mm, vias 0 -> 3
- net GND: track 0.00 -> 4.01 mm
- net CSB: track 0.00 -> 1.35 mm
- net footprint-cathode-0: track 0.00 -> 1.34 mm
- net footprint-cathode-1: track 0.00 -> 1.27 mm
- net MOSI: track 0.00 -> 1.18 mm
- net SCL: track 0.00 -> 1.11 mm
